File: Prinsip/Prinsip.sch (KiCad schematic (older format))
At the start: 1 part

Commit message: Initial prinsip
Parts:
- added U? (x4): 7410N, symbol Prinsip:7410N
- added U?: 74ALS21AM, symbol Prinsip:74ALS21AM
- added U?: 7432N, symbol Prinsip:7432N
- added U?: 7408J, symbol Prinsip:7408J
- added U? (x5): 7405N, symbol Prinsip:7405N
- added U?: 74157N, symbol Prinsip:74157N
- added U? (x2): 74F164D, symbol Prinsip:74F164D
Connections:
- new net: U?.2 (A), U?.3 (B), U?.4 (Qa)
- new net: U?.2 (A), U?.3 (B)
- new net GND: U?.8 (GND), U?.8 (GND), U?.8 (GND)
- new net Gnd: U?.7 (Gnd), U?.7 (Gnd), U?.7 (Gnd), U?.7 (Gnd), U?.7 (Gnd), U?.7 (Gnd), U?.7 (Gnd)
- new net VCC: U?.16 (VCC), U?.16 (VCC), U?.16 (VCC)
- new net Vcc: U?.14 (Vcc), U?.14 (Vcc), U?.14 (Vcc), U?.14 (Vcc), U?.14 (Vcc), U?.14 (Vcc), U?.14 (Vcc)
Changed lines of the file:
@@
 	1    0    0    -1
 $EndComp
+$Comp
+L Prinsip:7410N U?
+U 1 1 6166773C
+P 5850 3250
+F 0 "U?" H 5850 3666 50  0000 C CNN
+F 1 "7410N" H 5850 3575 50  0000 C CNN
+F 2 "" H 5850 3350 50  0001 C CNN
+F 3 "" H 5850 3350 50  0001 C CNN
+	1    5850 3250
+	1    0    0    -1
+$EndComp
+$Comp
+L Prinsip:74ALS21AM U?
+U 1 1 6166F230
+P 5850 2350
+F 0 "U?" H 5850 2766 50  0000 C CNN
+F 1 "74ALS21AM" H 5850 2675 50  0000 C CNN
+F 2 "" H 5850 2450 50  0001 C CNN
+F 3 "" H 5850 2450 50  0001 C CNN
+	1    5850 2350
+	1    0    0    -1
+$EndComp
+$Comp
+L Prinsip:7432N U?
+U 1 1 61674B22
+P 3300 2800
+F 0 "U?" H 3300 3216 50  0000 C CNN
+F 1 "7432N" H 3300 3125 50  0000 C CNN
+F 2 "" H 3300 2900 50  0001 C CNN
+F 3 "" H 3300 2900 50  0001 C CNN
+	1    3300 2800
+	1    0    0    -1
+$EndComp
+$Comp
+L Prinsip:7408J U?
+U 1 1 6167545D
+P 3300 3650
+F 0 "U?" H 3300 4066 50  0000 C CNN
+F 1 "7408J" H 3300 3975 50  0000 C CNN
+F 2 "" H 3300 3750 50  0001 C CNN
+F 3 "" H 3300 3750 50  0001 C CNN
+	1    3300 3650
+	1    0    0    -1
+$EndComp
+$Comp
+L Prinsip:7405N U?
+U 1 1 61675F5B
+P 7300 2350
+F 0 "U?" H 7300 2866 50  0000 C CNN
+F 1 "7405N" H 7300 2775 50  0000 C CNN
+F 2 "" H 7300 2550 50  0001 C CNN
+F 3 "" H 7300 2550 50  0001 C CNN
+	1    7300 2350
+	1    0    0    -1
+$EndComp
+$Comp
+L Prinsip:7405N U?
+U 1 1 61676BE0
+P 7300 3200
+F 0 "U?" H 7300 3716 50  0000 C CNN
+F 1 "7405N" H 7300 3625 50  0000 C CNN
+F 2 "" H 7300 3400 50  0001 C CNN
+F 3 "" H 7300 3400 50  0001 C CNN
+	1    7300 3200
+	1    0    0    -1
+$EndComp
+$Comp
+L Prinsip:7405N U?
+U 1 1 61677469
+P 7300 4050
+F 0 "U?" H 7300 4566 50  0000 C CNN
+F 1 "7405N" H 7300 4475 50  0000 C CNN
+F 2 "" H 7300 4250 50  0001 C CNN
+F 3 "" H 7300 4250 50  0001 C CNN
+	1    7300 4050
+	1    0    0    -1
+$EndComp
+$Comp
+L Prinsip:7410N U?
+U 1 1 616781C6
+P 8650 3600
+F 0 "U?" H 8650 4016 50  0000 C CNN
+F 1 "7410N" H 8650 3925 50  0000 C CNN
+F 2 "" H 8650 3700 50  0001 C CNN
+F 3 "" H 8650 3700 50  0001 C CNN
+	1    8650 3600
+	1    0    0    -1
+$EndComp
+$Comp
+L Prinsip:7410N U?
+U 1 1 616792E6
+P 8650 2900
+F 0 "U?" H 8650 3316 50  0000 C CNN
+F 1 "7410N" H 8650 3225 50  0000 C CNN
+F 2 "" H 8650 3000 50  0001 C CNN
+F 3 "" H 8650 3000 50  0001 C CNN
+	1    8650 2900
+	1    0    0    -1
+$EndComp
+$Comp
+L Prinsip:7405N U?
+U 1 1 61679C6F
+P 8650 2150
+F 0 "U?" H 8650 2666 50  0000 C CNN
+F 1 "7405N" H 8650 2575 50  0000 C CNN
+F 2 "" H 8650 2350 50  0001 C CNN
+F 3 "" H 8650 2350 50  0001 C CNN
+	1    8650 2150
+	1    0    0    -1
+$EndComp
+$Comp
+L Prinsip:7410N U?
+U 1 1 6167AB47
+P 10000 2900
+F 0 "U?" H 10000 3316 50  0000 C CNN
+F 1 "7410N" H 10000 3225 50  0000 C CNN
+F 2 "" H 10000 3000 50  0001 C CNN
+F 3 "" H 10000 3000 50  0001 C CNN
+	1    10000 2900
+	1    0    0    -1
+$EndComp
+$Comp
+L Prinsip:7405N U?
+U 1 1 6167B68A
+P 11200 3550
+F 0 "U?" H 11200 4066 50  0000 C CNN
+F 1 "7405N" H 11200 3975 50  0000 C CNN
+F 2 "" H 11200 3750 50  0001 C CNN
+F 3 "" H 11200 3750 50  0001 C CNN
+	1    11200 3550
+	1    0    0    -1
+$EndComp
+$Comp
+L Prinsip:74157N U?
+U 1 1 6167DF8D
+P 12350 2500
+F 0 "U?" H 12350 3216 50  0000 C CNN
+F 1 "74157N" H 12350 3125 50  0000 C CNN
+F 2 "" H 12400 3100 50  0001 C CNN
+F 3 "" H 12400 3100 50  0001 C CNN
+	1    12350 2500
+	1    0    0    -1
+$EndComp
+$Comp
+L Prinsip:74F164D U?
+U 1 1 616815DE
+P 13850 2500
+F 0 "U?" H 13850 3216 50  0000 C CNN
+F 1 "74F164D" H 13850 3125 50  0000 C CNN
+F 2 "" H 13900 3100 50  0001 C CNN
+F 3 "" H 13900 3100 50  0001 C CNN
+	1    13850 2500
+	1    0    0    -1
+$EndComp
+$Comp
+L Prinsip:74F164D U?
+U 1 1 61683A40
+P 13850 3950
+F 0 "U?" H 13850 4666 50  0000 C CNN
+F 1 "74F164D" H 13850 4575 50  0000 C CNN
+F 2 "" H 13900 4550 50  0001 C CNN
+F 3 "" H 13900 4550 50  0001 C CNN
+	1    13850 3950
+	1    0    0    -1
+$EndComp
+Wire Wire Line
+	13300 3800 13300 3900
+Wire Wire Line
+	13300 2350 13300 2450
+Wire Wire Line
+	12900 2350 13300 2350
+Connection ~ 13300 2350
 $EndSCHEMATC

Commit message: Updated princ
Parts:
- added U?: 74ALS11AM, symbol Prinsip:74ALS11AM
- added U?: 7405N, symbol Prinsip:7405N
Connections:
- net Gnd: now also U?.7 (Gnd)
- net Vcc: now also U?.14 (Vcc)
- net at U?.~ (~LOAD): now also U?.9
- net at U?.10: now also U?.~ (~LOAD)
- net at U?.12: now also U?.~ (~LOAD)
- net at U?.13: now also U?.~ (~LOAD)
- net at U?.8: now also U?.1
- net at U?.2: now also U?.2
- net at U?.2: now also U?.13, U?.2
- net at U?.2: now also U?.13
- net at U?.12: now also U?.13
- net at U?.12: now also U?.2
- net at U?.2: now also U?.1
- net at U?.12: now also U?.1, U?.2 (I0a)
- net at U?.2: now also U?.14 (I0v)
- net at U?.9 (Qh): now also U?.2 (A), U?.3 (B)
- new net: U?.1, U?.2
Other:
- note added: "CLK"
- note added: "SHIFT_CLR"
- moved on the sheet: U?, U?A

Commit message: Updated prinsip
Parts:
- added U? (x8): SW, symbol Prinsip:SW
Connections:
- net at U?.1: now also U?.9, U?.~ (~LOAD)
- net at U?.12: now also U?.2
- net at U?.13: now also U?.13, U?.~ (~LOAD)
- net at U?.2: now also U?.10, U?.~ (~LOAD)
- net at U?.~ (~LOAD): now also U?.~
- net at U?.1, U?.8: now also U?.1
- net at U?.2: now also U?.3
- net at U?.3: now also U?.~ (~LOAD)
- net at U?.1: now also U?.~
- net at U?.9 (Qh): now also U?.2 (A), U?.3 (B)
Other:
- note added: "GND"
- note added: "VCC"
- moved on the sheet: U?, U?A

Commit message: Updated
Connections:
- net RCO: now reaches U?.~ (~LOAD)
- net at U?.12: no longer U?.~ (~LOAD)
- net at U?.~: no longer U?.~ (~LOAD)
- net at U?.1, U?.8: no longer U?.1
- net at U?.9 (Qh): now also U?.2 (A), U?.3 (B)
- new net: U?.~, U?.~ (~LOAD)
- now unconnected: U?.1, U?.10, U?.13, U?.13, U?.2, U?.9
Other:
- note added: "SW1"
Changed lines of the file:
@@
 	8350 1300 8350 1400
 Wire Bus Line
-	9450 1850 9450 1600
-Wire Bus Line
 	8200 1850 9450 1850
-Entry Wire Line
-	9350 1500 9450 1600
-Wire Wire Line
-	5700 2250 5300 2250
-Wire Wire Line
-	5300 2250 5300 2900
-Wire Wire Line
-	5300 2900 5200 2900
-Wire Wire Line
-	5200 3000 5400 3000
-Wire Wire Line
-	5400 3000 5400 2350
-Wire Wire Line
-	5400 2350 5700 2350
-Wire Wire Line
-	5700 2450 5500 2450
-Wire Wire Line
-	5500 2450 5500 3100
-Wire Wire Line
-	5500 3100 5200 3100
-Wire Wire Line
-	5200 3200 5500 3200
-Wire Wire Line
-	5600 3200 5600 2550
-Wire Wire Line
-	5600 2550 5700 2550
 Wire Wire Line
 	6700 2350 6800 2350
 Wire Wire Line
-	6800 2350 6800 1750
-Wire Wire Line
-	6800 1300 7050 1300
-Wire Wire Line
-	5300 2900 5900 2900
-Wire Wire Line
-	5900 2900 5900 3500
-Connection ~ 5300 2900
-Wire Wire Line
-	5400 3000 5800 3000
-Wire Wire Line
-	5800 3000 5800 3600
-Wire Wire Line
-	5800 3600 5900 3600
-Connection ~ 5400 3000
-Wire Wire Line
-	5500 3200 5500 3700
-Wire Wire Line
-	5500 3700 5900 3700
-Connection ~ 5500 3200
-Wire Wire Line
-	5500 3200 5600 3200
-Wire Wire Line
 	4300 3550 4400 3550
 Wire Wire Line
 	3050 3650 3200 3650
-Wire Wire Line
-	3200 3450 3200 1750
-Wire Wire Line
-	3200 1750 6800 1750
-Connection ~ 6800 1750
-Wire Wire Line
-	6800 1750 6800 1300
 $Comp
 L Prinsip:SW U?
@@
 	4300 3650 4400 3650
 Wire Bus Line
+	1100 900  1750 900
+Wire Bus Line
+	6450 900  6450 400
+Wire Bus Line
+	6450 400  6800 400
+Connection ~ 9450 400
+Wire Bus Line
+	9450 400  16050 400
+Entry Wire Line
+	9350 1500 9450 1600
+Connection ~ 1750 900
+Wire Bus Line
+	1750 900  3100 900
+Entry Wire Line
+	1650 2700 1750 2800
+Entry Wire Line
+	1650 3000 1750 3100
+Entry Wire Line
+	1650 3300 1750 3400
+Entry Wire Line
+	1650 3600 1750 3700
+Entry Wire Line
+	1650 3900 1750 4000
+Entry Wire Line
+	1650 4200 1750 4300
+Wire Wire Line
+	6800 1300 6800 2350
+Connection ~ 3100 900
+Wire Bus Line
+	3100 900  5550 900
+Entry Wire Line
+	3100 3350 3200 3450
+Wire Bus Line
+	6800 400  6800 1200
+Connection ~ 6800 400
+Wire Bus Line
+	6800 400  9450 400
+Entry Wire Line
+	6800 1200 6900 1300
+Entry Bus Bus
+	3100 2400 3200 2500
+Wire Bus Line
+	3200 2500 4150 2500
+Entry Wire Line
+	4150 2800 4250 2900
+Entry Wire Line
+	4150 2900 4250 3000
+Entry Wire Line
+	4150 3000 4250 3100
+Entry Wire Line
+	4150 3100 4250 3200
+Entry Wire Line
+	4150 3250 4250 3350
+Entry Wire Line
+	4150 3350 4250 3450
+Wire Wire Line
+	4250 2900 4400 2900
+Text Notes 4250 2900 0    50   ~ 0
+SW1
+Wire Wire Line
+	4250 3000 4400 3000
+Wire Wire Line
+	4250 3100 4400 3100
+Wire Wire Line
+	4400 3200 4250 3200
+Wire Wire Line
+	4250 3350 4400 3350
+Wire Wire Line
+	4400 3450 4250 3450
+Connection ~ 5550 900
+Wire Bus Line
+	5550 900  6450 900
+Wire Wire Line
+	5200 2900 5450 2900
+Entry Wire Line
+	5450 2900 5550 3000
+Wire Wire Line
+	5200 3000 5450 3000
+Entry Wire Line
+	5450 3000 5550 3100
+Wire Wire Line
+	5200 3100 5450 3100
+Entry Wire Line
+	5450 3100 5550 3200
+Wire Wire Line
+	5200 3200 5450 3200
+Entry Wire Line
+	5450 3200 5550 3300
+Text GLabel 5250 3300 2    50   Input ~ 0
+RCO
+Wire Wire Line
+	5200 3300 5250 3300
+Wire Wire Line
+	5650 2250 5700 2250
+Wire Wire Line
+	5650 2350 5700 2350
+Entry Wire Line
+	5550 2150 5650 2250
+Entry Wire Line
+	5550 2250 5650 2350
+Entry Wire Line
+	5550 2350 5650 2450
+Entry Wire Line
+	5550 2450 5650 2550
+Wire Wire Line
+	5650 2450 5700 2450
+Wire Wire Line
+	5700 2550 5650 2550
+Wire Wire Line
+	5650 3500 5900 3500
+Wire Wire Line
+	5900 3600 5650 3600
+Wire Wire Line
+	5650 3700 5900 3700
+Wire Bus Line
+	3100 900  3100 3350
+Wire Wire Line
+	6800 1300 7050 1300
+Wire Bus Line
+	9450 400  9450 1850
+Wire Bus Line
 	8200 1400 8200 1850
 Wire Bus Line
 	13500 5550 13500 8100
 Wire Bus Line
+	1750 900  1750 4300
+Wire Bus Line
+	4150 2500 4150 3400
+Wire Bus Line
+	5550 900  5550 3750
+Wire Bus Line
 	15250 4700 15250 8100
 Wire Bus Line
-	1100 2500 1100 5000
+	1100 900  1100 5000
+Entry Wire Line
+	5550 3400 5650 3500
+Entry Wire Line
+	5550 3500 5650 3600
+Entry Wire Line
+	5550 3600 5650 3700
 $EndSCHEMATC

Commit message: Updated
Parts:
- added BAR?: HDSP-4830_2, Display:HDSP-4830, symbol Prinsip:HDSP-4830_2
- added BAR?: HDSP-4830_2_copy, Display:HDSP-4830, symbol Prinsip:HDSP-4830_2_copy
- added U? (x2): 74273DW, symbol Prinsip:74273DW
- added U?: 7405N, symbol Prinsip:7405N
Connections:
- net GND: now also U?.8 (GND), U?.8 (GND)
- net VCC: now also U?.16 (VCC), U?.16 (VCC)
- net QB: now reaches U?.1
- net QB: now also U?.1, U?.12, U?.~ (~LOAD)
- net QD: now reaches U?.13
- net QD: now also U?.1, U?.9, U?.~ (~LOAD)
- net QA: now reaches U?.2
- net QA: now also U?.1, U?.1, U?.13, U?.~ (~LOAD)
- net at U?.~: no longer U?.~ (~LOAD)
- net QC: now reaches U?.10
- net QC: now also U?.1, U?.1, U?.~ (~LOAD)
- net at U?.9 (Qh): now also U?.2 (A), U?.3 (B)
- new net: U?.~, U?.~ (~LOAD)
- new net: U?.1 (CLK), U?.1 (CLK), U?.2
- new net: BAR?.3 (A), U?.12 (7Q) (x2)
- new net: BAR?.7 (A), U?.12 (7Q)
- new net: BAR?.1 (A), U?.4 (5Q) (x2)
- new net: BAR?.5 (A), U?.4 (5Q)
- new net: BAR?.2 (A), U?.7 (6Q) (x2)
- new net: BAR?.6 (A), U?.7 (6Q)
- new net: BAR?.4 (A), U?.9 (8Q)
- new net: BAR?.8 (A), U?.9 (8Q)
- new net: BAR?.13 (K), BAR?.14 (K), BAR?.15 (K), BAR?.16 (K), BAR?.17 (K), BAR?.18 (K), BAR?.19 (K), BAR?.20 (K)
- new net: BAR?.18 (K), BAR?.19 (K), BAR?.20 (K)
- new net +5V: U?.15 (~CLR), U?.15 (~CLR)
- new net Q0: U?.2 (1D)
- new net Q1: U?.3 (2D)
- new net Q10: U?.5 (3D)
- new net Q2: U?.5 (3D)
- new net Q3: U?.6 (4D)
- new net Q4: U?.14 (5D)
- new net Q5: U?.13 (6D)
- new net Q6: U?.11 (7D)
- new net Q7: U?.10 (8D)
- new net Q8: U?.2 (1D)
- new net Q9: U?.3 (2D)
- new net TO_BUFFER: U?.1
Other:
- moved on the sheet: U?A
Changed lines of the file:
@@
 L Prinsip:7410N U?
 U 1 1 6166773C
-P 6400 3600
-F 0 "U?" H 6400 4016 50  0000 C CNN
-F 1 "7410N" H 6400 3925 50  0000 C CNN
-F 2 "" H 6400 3700 50  0001 C CNN
-F 3 "" H 6400 3700 50  0001 C CNN
-	1    6400 3600
-	1    0    0    -1
-$EndComp
-$Comp
-L Prinsip:74ALS21AM U?
-U 1 1 6166F230
-P 6200 2350
-F 0 "U?" H 6200 2766 50  0000 C CNN
-F 1 "74ALS21AM" H 6200 2675 50  0000 C CNN
-F 2 "" H 6200 2450 50  0001 C CNN
-F 3 "" H 6200 2450 50  0001 C CNN
-	1    6200 2350
+P 6200 3600
+F 0 "U?" H 6200 4016 50  0000 C CNN
+F 1 "7410N" H 6200 3925 50  0000 C CNN
+F 2 "" H 6200 3700 50  0001 C CNN
+F 3 "" H 6200 3700 50  0001 C CNN
+	1    6200 3600
 	1    0    0    -1
 $EndComp
@@
 GND
 Wire Wire Line
-	6900 3600 6900 4000
-Wire Wire Line
-	6900 4000 1950 4000
+	6700 3600 6700 4000
 Wire Wire Line
 	1950 4000 1950 3750
@@
 	6800 1300 6800 2350
 Connection ~ 3100 900
-Wire Bus Line
-	3100 900  5550 900
 Entry Wire Line
 	3100 3350 3200 3450
@@
 Wire Wire Line
 	4400 3450 4250 3450
-Connection ~ 5550 900
-Wire Bus Line
-	5550 900  6450 900
-Wire Wire Line
-	5200 2900 5450 2900
-Entry Wire Line
-	5450 2900 5550 3000
-Wire Wire Line
-	5200 3000 5450 3000
-Entry Wire Line
-	5450 3000 5550 3100
-Wire Wire Line
-	5200 3100 5450 3100
-Entry Wire Line
-	5450 3100 5550 3200
-Wire Wire Line
-	5200 3200 5450 3200
-Entry Wire Line
-	5450 3200 5550 3300
 Text GLabel 5250 3300 2    50   Input ~ 0
 RCO
 Wire Wire Line
 	5200 3300 5250 3300
-Wire Wire Line
-	5650 2250 5700 2250
-Wire Wire Line
-	5650 2350 5700 2350
-Entry Wire Line
-	5550 2150 5650 2250
-Entry Wire Line
-	5550 2250 5650 2350
-Entry Wire Line
-	5550 2350 5650 2450
-Entry Wire Line
-	5550 2450 5650 2550
-Wire Wire Line
-	5650 2450 5700 2450
-Wire Wire Line
-	5700 2550 5650 2550
-Wire Wire Line
-	5650 3500 5900 3500
-Wire Wire Line
-	5900 3600 5650 3600
-Wire Wire Line
-	5650 3700 5900 3700
+Wire Bus Line
+	3100 900  6450 900
+$Comp
+L Prinsip:74ALS21AM U?
+U 1 1 6166F230
+P 6200 2350
+F 0 "U?" H 6200 2766 50  0000 C CNN
+F 1 "74ALS21AM" H 6200 2675 50  0000 C CNN
+F 2 "" H 6200 2450 50  0001 C CNN
+F 3 "" H 6200 2450 50  0001 C CNN
+	1    6200 2350
+	1    0    0    -1
+$EndComp
+Text GLabel 5300 2900 2    50   Input ~ 0
+QA
+Text GLabel 5300 3000 2    50   Input ~ 0
+QB
+Text GLabel 5300 3100 2    50   Input ~ 0
+QC
+Text GLabel 5300 3200 2    50   Input ~ 0
+QD
+Wire Wire Line
+	5200 2900 5300 2900
+Wire Wire Line
+	5300 3000 5200 3000
+Wire Wire Line
+	5200 3100 5300 3100
+Wire Wire Line
+	5300 3200 5200 3200
+Text GLabel 5600 2550 0    50   Input ~ 0
+QA
+Text GLabel 5600 2450 0    50   Input ~ 0
+QB
+Text GLabel 5600 2350 0    50   Input ~ 0
+QC
+Text GLabel 5600 2250 0    50   Input ~ 0
+QD
+Wire Wire Line
+	5600 2250 5700 2250
+Wire Wire Line
+	5700 2350 5600 2350
+Wire Wire Line
+	5600 2450 5700 2450
+Wire Wire Line
+	5700 2550 5600 2550
+Text GLabel 5700 3600 0    50   Input ~ 0
+QA
+Text GLabel 5700 3500 0    50   Input ~ 0
+QB
+Text GLabel 5700 3700 0    50   Input ~ 0
+QD
+Wire Wire Line
+	6700 4000 1950 4000
+Text GLabel 7000 5500 0    50   Input ~ 0
+QA
+Text GLabel 7000 6350 0    50   Input ~ 0
+QB
+Text GLabel 7000 7200 0    50   Input ~ 0
+QC
+Text GLabel 8850 4900 0    50   Input ~ 0
+QD
+Text GLabel 8450 5400 0    50   Input ~ 0
+QC
+Text GLabel 8900 6000 0    50   Input ~ 0
+QA
+$Comp
+L Prinsip:74273DW U?
+U 1 1 618BBFDD
+P 11800 1600
+F 0 "U?" H 11800 2316 50  0000 C CNN
+F 1 "74273DW" H 11800 2225 50  0000 C CNN
+F 2 "" H 11850 2200 50  0001 C CNN
+F 3 "" H 11850 2200 50  0001 C CNN
+	1    11800 1600
+	1    0    0    -1
+$EndComp
+$Comp
+L Prinsip:74273DW U?
+U 1 1 618BD466
+P 11800 3200
+F 0 "U?" H 11800 3916 50  0000 C CNN
+F 1 "74273DW" H 11800 3825 50  0000 C CNN
+F 2 "" H 11850 3800 50  0001 C CNN
+F 3 "" H 11850 3800 50  0001 C CNN
+	1    11800 3200
+	1    0    0    -1
+$EndComp
+Text GLabel 11250 1200 0    50   Input ~ 0
+Q0
+Text GLabel 11250 1300 0    50   Input ~ 0
+Q1
+Text GLabel 11250 1400 0    50   Input ~ 0
+Q2
+Text GLabel 11250 1500 0    50   Input ~ 0
+Q3
+Text GLabel 11250 1600 0    50   Input ~ 0
+Q4
+Text GLabel 11250 1700 0    50   Input ~ 0
+Q5
+Text GLabel 11250 1800 0    50   Input ~ 0
+Q6
+Text GLabel 11250 1900 0    50   Input ~ 0
+Q7
+Text GLabel 11250 2800 0    50   Input ~ 0
+Q8
+Text GLabel 11250 2900 0    50   Input ~ 0
+Q9
+Text GLabel 11250 3000 0    50   Input ~ 0
+Q10
+Text GLabel 11250 2100 0    50   Input ~ 0
++5V
+Text GLabel 11250 3700 0    50   Input ~ 0
++5V
+Wire Wire Line
+	11250 2200 10850 2200
+Wire Wire Line
+	10850 2200 10850 3000
+Wire Wire Line
+	10850 3800 11250 3800
+$Comp
+L Prinsip:7405N U?
+U 1 1 618EAB2F
+P 10300 3000
+F 0 "U?" H 10300 3516 50  0000 C CNN
+F 1 "7405N" H 10300 3425 50  0000 C CNN
+F 2 "" H 10300 3200 50  0001 C CNN
+F 3 "" H 10300 3200 50  0001 C CNN
+	1    10300 3000
+	1    0    0    -1
+$EndComp
+Connection ~ 10850 3000
+Wire Wire Line
+	10850 3000 10850 3800
+Text GLabel 9750 3000 0    50   Input ~ 0
+TO_BUFFER
+$Comp
+L Prinsip:HDSP-4830_2 BAR?
+U 1 1 6190A90C
+P 12550 1600
+F 0 "BAR?" H 12550 2175 50  0001 C CNN
+F 1 "HDSP-4830_2" H 12550 2176 50  0001 C CNN
+F 2 "Display:HDSP-4830" H 12550 800 50  0001 C CNN
+F 3 "https://docs.broadcom.com/docs/AV02-1798EN" H 10550 1800 50  0001 C CNN
+	1    12550 1600
+	1    0    0    -1
+$EndComp
+Wire Wire Line
+	12750 1200 12850 1200
+Wire Wire Line
+	12850 1200 12850 1300
+$Comp
+L Prinsip:HDSP-4830_2_copy BAR?
+U 1 1 619249F3
+P 12550 3200
+F 0 "BAR?" H 12550 3867 50  0000 C CNN
+F 1 "HDSP-4830_2_copy" H 12550 3776 50  0000 C CNN
+F 2 "Display:HDSP-4830" H 12550 2400 50  0001 C CNN
+F 3 "https://docs.broadcom.com/docs/AV02-1798EN" H 10550 3400 50  0001 C CNN
+	1    12550 3200
+	1    0    0    -1
+$EndComp
+Wire Wire Line
+	12750 2800 12850 2800
+Wire Wire Line
+	12850 2800 12850 2900
+Wire Wire Line
+	12750 2900 12850 2900
+Connection ~ 12850 2900
+Wire Wire Line
+	12850 2900 12850 3000
+Wire Wire Line
+	12750 3000 12850 3000
+Connection ~ 12850 3000
+Wire Wire Line
+	12850 3000 12850 3050
+Wire Wire Line
+	12750 1300 12850 1300
+Connection ~ 12850 1300
+Wire Wire Line
+	12850 1300 12850 1400
+Wire Wire Line
+	12750 1400 12850 1400
+Connection ~ 12850 1400
+Wire Wire Line
+	12850 1400 12850 1500
+Wire Wire Line
+	12750 1500 12850 1500
+Connection ~ 12850 1500
+Wire Wire Line
+	12850 1500 12850 1600
+Wire Wire Line
+	12750 1600 12850 1600
+Connection ~ 12850 1600
+Wire Wire Line
+	12850 1600 12850 1700
+Wire Wire Line
+	12750 1700 12850 1700
+Connection ~ 12850 1700
+Wire Wire Line
+	12850 1700 12850 1800
+Wire Wire Line
+	12750 1800 12850 1800
+Connection ~ 12850 1800
+Wire Wire Line
+	12850 1800 12850 1900
+Wire Wire Line
+	12750 1900 12850 1900
 Wire Bus Line
 	3100 900  3100 3350
@@
 	4150 2500 4150 3400
 Wire Bus Line
-	5550 900  5550 3750
-Wire Bus Line
 	15250 4700 15250 8100
 Wire Bus Line
 	1100 900  1100 5000
-Entry Wire Line
-	5550 3400 5650 3500
-Entry Wire Line
-	5550 3500 5650 3600
-Entry Wire Line
-	5550 3600 5650 3700
+Connection ~ 12850 1900
+Wire Wire Line
+	12850 1900 12850 1950
 $EndSCHEMATC

Commit message: Updated
Parts:
- added U?: 74163N, symbol Prinsip:74163N
- added U?: 74F164D, symbol Prinsip:74F164D
- added U?: 4512BD, symbol 4xxx_IEEE:4512
- added U?: 7402, symbol 74xx_IEEE:7402
- added U?: 7474N, symbol Prinsip:7474N
Connections:
- net +5V: now also U?.2
- net GND: now also U?.4 (GND), U?.7 (GND), U?.8 (GND)
- net VCC: now also U?.14 (VCC), U?.16 (VCC), U?.8 (VCC)
- net at U?.~: no longer U?.~ (~LOAD)
- net at U?.9 (Qh): now also U?.2 (A), U?.3 (B)
- net at U?.12 (7Q): now also BAR?.3 (A)
- net at U?.4 (5Q): now also BAR?.1 (A)
- net at U?.7 (6Q): now also BAR?.2 (A)
- net Earth: now reaches BAR?.13 (K), BAR?.14 (K), BAR?.15 (K), BAR?.16 (K), BAR?.17 (K), BAR?.18 (K), BAR?.19 (K), BAR?.20 (K)
- net Earth: now also BAR?.18 (K), BAR?.19 (K), BAR?.20 (K)
- new net: U?.~, U?.~ (~LOAD)
- new net: U?.2 (A), U?.3 (B), U?.~ (~LOAD)
- new net: U?.12 (Qg), U?.3 (I2)
- new net: U?.12 (Qg), U?.7 (I6)
- new net: U?.1 (I0), U?.4 (Qe)
- new net: U?.4 (Qe), U?.5 (I4)
- new net: U?.2 (I1), U?.7 (Qf)
- new net: U?.6 (I5), U?.7 (Qf)
- new net: U?.4 (I3), U?.9 (Qh)
- new net: U?.9 (I7), U?.9 (Qh)
- new net QC1: U?.3, U?.~ (~LOAD)
- new net Vdd: U?.16 (Vdd)
- new net Vss: U?.8 (Vss)
Changed lines of the file:
@@
 Wire Wire Line
 	12750 1900 12850 1900
+Connection ~ 12850 1900
+Wire Wire Line
+	12850 1900 12850 1950
+$Comp
+L power:Earth #PWR?
+U 1 1 6196B4C4
+P 12850 1950
+F 0 "#PWR?" H 12850 1700 50  0001 C CNN
+F 1 "Earth" H 12850 1800 50  0001 C CNN
+F 2 "" H 12850 1950 50  0001 C CNN
+F 3 "~" H 12850 1950 50  0001 C CNN
+	1    12850 1950
+	1    0    0    -1
+$EndComp
+$Comp
+L power:Earth #PWR?
+U 1 1 6196C1EF
+P 12850 3050
+F 0 "#PWR?" H 12850 2800 50  0001 C CNN
+F 1 "Earth" H 12850 2900 50  0001 C CNN
+F 2 "" H 12850 3050 50  0001 C CNN
+F 3 "~" H 12850 3050 50  0001 C CNN
+	1    12850 3050
+	1    0    0    -1
+$EndComp
+$Comp
+L Prinsip:74163N U?
+U 1 1 6196D97B
+P 2800 9300
+F 0 "U?" H 2850 9365 50  0000 C CNN
+F 1 "74163N" H 2850 9274 50  0000 C CNN
+F 2 "" H 2800 9300 50  0001 C CNN
+F 3 "" H 2800 9300 50  0001 C CNN
+	1    2800 9300
+	1    0    0    -1
+$EndComp
+$Comp
+L Prinsip:74F164D U?
+U 1 1 6196E84B
+P 4800 9650
+F 0 "U?" H 4800 10366 50  0000 C CNN
+F 1 "74F164D" H 4800 10275 50  0000 C CNN
+F 2 "" H 4850 10250 50  0001 C CNN
+F 3 "" H 4850 10250 50  0001 C CNN
+	1    4800 9650
+	1    0    0    -1
+$EndComp
+$Comp
+L 4xxx_IEEE:4512 U?
+U 1 1 6196F3A5
+P 6350 9500
+F 0 "U?" H 6350 10366 50  0000 C CNN
+F 1 "4512BD" H 6350 10275 50  0000 C CNN
+F 2 "" H 6350 9500 50  0001 C CNN
+F 3 "" H 6350 9500 50  0001 C CNN
+	1    6350 9500
+	1    0    0    -1
+$EndComp
+Wire Wire Line
+	5350 9400 5800 9400
+Wire Wire Line
+	5800 9500 5350 9500
+Wire Wire Line
+	5350 9600 5800 9600
+Wire Wire Line
+	5800 9700 5350 9700
+Wire Wire Line
+	5350 9800 5800 9800
+Wire Wire Line
+	5800 9900 5350 9900
+Wire Wire Line
+	5350 10000 5800 10000
+Wire Wire Line
+	5800 10100 5350 10100
+Wire Wire Line
+	4250 9600 4250 9500
+Wire Wire Line
+	3250 9500 4250 9500
+Connection ~ 4250 9500
+$Comp
+L 74xx_IEEE:7402 U?
+U 1 1 619CFB28
+P 3950 8350
+F 0 "U?" H 3950 8816 50  0000 C CNN
+F 1 "7402" H 3950 8725 50  0000 C CNN
+F 2 "" H 3950 8350 50  0001 C CNN
+F 3 "" H 3950 8350 50  0001 C CNN
+	1    3950 8350
+	1    0    0    -1
+$EndComp
+$Comp
+L Prinsip:7474N U?
+U 1 1 619D0C4B
+P 4750 6950
+F 0 "U?" H 4750 7381 50  0000 C CNN
+F 1 "7474N" H 4750 7290 50  0000 C CNN
+F 2 "" H 4750 6950 50  0001 C CNN
+F 3 "http://www.ti.com/lit/sg/scyt129e/scyt129e.pdf" H 4750 6950 50  0001 C CNN
+	1    4750 6950
+	1    0    0    -1
+$EndComp
+Text GLabel 3400 8450 0    50   Input ~ 0
+QC1
+Text GLabel 3250 9700 2    50   Input ~ 0
+QC1
 Wire Bus Line
 	3100 900  3100 3350
@@
 Wire Bus Line
 	1100 900  1100 5000
-Connection ~ 12850 1900
-Wire Wire Line
-	12850 1900 12850 1950
+$Comp
+L power:+5V #PWR?
+U 1 1 61A21106
+P 3400 8250
+F 0 "#PWR?" H 3400 8100 50  0001 C CNN
+F 1 "+5V" H 3415 8423 50  0000 C CNN
+F 2 "" H 3400 8250 50  0001 C CNN
+F 3 "" H 3400 8250 50  0001 C CNN
+	1    3400 8250
+	1    0    0    -1
+$EndComp
 $EndSCHEMATC
