File: Prinsip/Prinsip.sch (KiCad schematic (older format))
At the start: 36 parts

Commit message: Updated
Parts:
- removed U?: 7402, symbol 74xx_IEEE:7402
- added U?: 74163N, symbol Prinsip:74163N
- added U? (x2): 7405N, symbol Prinsip:7405N
- added U?: 7402N, symbol Prinsip:7402N
- U?: value SW -> S8
- U?: value SW -> S7
- U?: value SW -> S6
- U?: value SW -> S5
- U?: value SW -> S4
- U?: value SW -> S3
- U?: value SW -> S2
- U?: value SW -> S1
Connections:
- net +5V: now also U?.2, U?.~ (~LOAD)
- net Earth: now also U?.10 (~E), U?.15 (~EN)
- net GND: now also U?.7 (GND)
- net QC1: now also U?.3
- net TO_BUFFER: now also U?.~ (~LOAD)
- net VCC: now also U?.14 (VCC)
- net at U?.~: no longer U?.~ (~LOAD)
- net QT: now reaches U?.1 (A/B)
- net QT: now also U?.5 (Q)
- net at U?.15 (~G): now also U?.1
- net at U?.9 (Qh): now also U?.2 (A), U?.3 (B)
- net at U?.12 (7Q): now also BAR?.3 (A)
- net at U?.4 (5Q): now also BAR?.1 (A)
- net at U?.7 (6Q): now also BAR?.2 (A)
- net at U?.1 (CLK): now also U?.2
- net at U?.11 (S0): now also U?.~ (~LOAD)
- net at U?.12 (S1): now also U?.~ (~LOAD)
- net at U?.13 (S2): now also U?.~ (~LOAD)
- net at U?.14 (Q): now also U?.2 (D)
- net at U?.1 (C): now also U?.2
- new net: U?.~, U?.~ (~LOAD)
- new net: U?.1, U?.~ (~LOAD)
- new net TO_BUFFER_1: U?.1
Other:
- moved on the sheet: U?
Changed lines of the file:
@@
 	12400 5500 12550 5500
 Wire Wire Line
-	12550 5100 12350 5100
-Wire Wire Line
-	12350 5100 12350 4750
-Wire Wire Line
-	12350 4750 11300 4750
-Wire Wire Line
-	11300 4750 11300 5500
+	12200 5100 12200 4900
 Wire Wire Line
 	11200 5500 11300 5500
@@
 P 1500 2550
 F 0 "U?" H 1500 2717 50  0001 C CNN
-F 1 "SW" H 1500 2625 50  0000 C CNN
+F 1 "S8" H 1500 2625 50  0000 C CNN
 F 2 "" H 1500 2550 50  0001 C CNN
 F 3 "" H 1500 2550 50  0001 C CNN
@@
 P 1500 2850
 F 0 "U?" H 1500 3017 50  0001 C CNN
-F 1 "SW" H 1500 2925 50  0000 C CNN
+F 1 "S7" H 1500 2925 50  0000 C CNN
 F 2 "" H 1500 2850 50  0001 C CNN
 F 3 "" H 1500 2850 50  0001 C CNN
@@
 P 1500 3150
 F 0 "U?" H 1500 3317 50  0001 C CNN
-F 1 "SW" H 1500 3225 50  0000 C CNN
+F 1 "S6" H 1500 3225 50  0000 C CNN
 F 2 "" H 1500 3150 50  0001 C CNN
 F 3 "" H 1500 3150 50  0001 C CNN
@@
 P 1500 3450
 F 0 "U?" H 1500 3617 50  0001 C CNN
-F 1 "SW" H 1500 3525 50  0000 C CNN
+F 1 "S5" H 1500 3525 50  0000 C CNN
 F 2 "" H 1500 3450 50  0001 C CNN
 F 3 "" H 1500 3450 50  0001 C CNN
@@
 P 1500 3750
 F 0 "U?" H 1500 3917 50  0001 C CNN
-F 1 "SW" H 1500 3825 50  0000 C CNN
+F 1 "S4" H 1500 3825 50  0000 C CNN
 F 2 "" H 1500 3750 50  0001 C CNN
 F 3 "" H 1500 3750 50  0001 C CNN
@@
 P 1500 4050
 F 0 "U?" H 1500 4217 50  0001 C CNN
-F 1 "SW" H 1500 4125 50  0000 C CNN
+F 1 "S3" H 1500 4125 50  0000 C CNN
 F 2 "" H 1500 4050 50  0001 C CNN
 F 3 "" H 1500 4050 50  0001 C CNN
@@
 P 1500 4350
 F 0 "U?" H 1500 4517 50  0001 C CNN
-F 1 "SW" H 1500 4425 50  0000 C CNN
+F 1 "S2" H 1500 4425 50  0000 C CNN
 F 2 "" H 1500 4350 50  0001 C CNN
 F 3 "" H 1500 4350 50  0001 C CNN
@@
 P 1500 4650
 F 0 "U?" H 1500 4817 50  0001 C CNN
-F 1 "SW" H 1500 4725 50  0000 C CNN
+F 1 "S1" H 1500 4725 50  0000 C CNN
 F 2 "" H 1500 4650 50  0001 C CNN
 F 3 "" H 1500 4650 50  0001 C CNN
@@
 Connection ~ 4250 9500
 $Comp
-L 74xx_IEEE:7402 U?
-U 1 1 619CFB28
-P 3950 8350
-F 0 "U?" H 3950 8816 50  0000 C CNN
-F 1 "7402" H 3950 8725 50  0000 C CNN
-F 2 "" H 3950 8350 50  0001 C CNN
-F 3 "" H 3950 8350 50  0001 C CNN
-	1    3950 8350
-	1    0    0    -1
-$EndComp
-$Comp
 L Prinsip:7474N U?
 U 1 1 619D0C4B
-P 4750 6950
-F 0 "U?" H 4750 7381 50  0000 C CNN
-F 1 "7474N" H 4750 7290 50  0000 C CNN
-F 2 "" H 4750 6950 50  0001 C CNN
-F 3 "http://www.ti.com/lit/sg/scyt129e/scyt129e.pdf" H 4750 6950 50  0001 C CNN
-	1    4750 6950
-	1    0    0    -1
-$EndComp
-Text GLabel 3400 8450 0    50   Input ~ 0
-QC1
+P 7400 9600
+F 0 "U?" H 7400 10031 50  0000 C CNN
+F 1 "7474N" H 7400 9940 50  0000 C CNN
+F 2 "" H 7400 9600 50  0001 C CNN
+F 3 "http://www.ti.com/lit/sg/scyt129e/scyt129e.pdf" H 7400 9600 50  0001 C CNN
+	1    7400 9600
+	1    0    0    -1
+$EndComp
 Text GLabel 3250 9700 2    50   Input ~ 0
 QC1
+$Comp
+L Prinsip:74163N U?
+U 1 1 61A3EC68
+P 4800 7700
+F 0 "U?" H 4850 7765 50  0000 C CNN
+F 1 "74163N" H 4850 7674 50  0000 C CNN
+F 2 "" H 4800 7700 50  0001 C CNN
+F 3 "" H 4800 7700 50  0001 C CNN
+	1    4800 7700
+	1    0    0    -1
+$EndComp
+Wire Wire Line
+	5250 7900 5650 7900
+Wire Wire Line
+	5650 7900 5650 9100
+Wire Wire Line
+	5650 9100 5800 9100
+Wire Wire Line
+	5250 8000 5550 8000
+Wire Wire Line
+	5550 8000 5550 9200
+Wire Wire Line
+	5550 9200 5800 9200
+Wire Wire Line
+	5250 8100 5450 8100
+Wire Wire Line
+	5450 8100 5450 9300
+Wire Wire Line
+	5450 9300 5800 9300
+Wire Wire Line
+	4450 8650 4350 8650
+Wire Wire Line
+	4350 8650 4350 8550
+Wire Wire Line
+	4350 7900 4450 7900
+Wire Wire Line
+	4450 8000 4350 8000
+Connection ~ 4350 8000
+Wire Wire Line
+	4350 8000 4350 7900
+Wire Wire Line
+	4450 8100 4350 8100
+Connection ~ 4350 8100
+Wire Wire Line
+	4350 8100 4350 8000
+Wire Wire Line
+	4450 8200 4350 8200
+Connection ~ 4350 8200
+Wire Wire Line
+	4350 8200 4350 8100
+Wire Wire Line
+	4450 8350 4350 8350
+Connection ~ 4350 8350
+Wire Wire Line
+	4350 8350 4350 8200
+Wire Wire Line
+	4450 8450 4350 8450
+Connection ~ 4350 8450
+Wire Wire Line
+	4350 8450 4350 8350
+Wire Wire Line
+	4450 8550 4350 8550
+Connection ~ 4350 8550
+Wire Wire Line
+	4350 8550 4350 8450
+Text GLabel 4350 7800 1    50   Input ~ 0
++5V
+Connection ~ 4350 7900
+Wire Wire Line
+	4350 7800 4350 7900
+Text GLabel 4450 8750 0    50   Input ~ 0
+TO_BUFFER
+$Comp
+L power:Earth #PWR?
+U 1 1 61AD2B5F
+P 5750 8700
+F 0 "#PWR?" H 5750 8450 50  0001 C CNN
+F 1 "Earth" H 5750 8550 50  0001 C CNN
+F 2 "" H 5750 8700 50  0001 C CNN
+F 3 "~" H 5750 8700 50  0001 C CNN
+	1    5750 8700
+	-1   0    0    1
+$EndComp
+Wire Wire Line
+	5800 9000 5750 9000
+Wire Wire Line
+	5750 9000 5750 8900
+Wire Wire Line
+	5800 8900 5750 8900
+Connection ~ 5750 8900
+Wire Wire Line
+	5750 8900 5750 8700
+$Comp
+L Prinsip:7405N U?
+U 1 1 61B006B1
+P 3650 10850
+F 0 "U?" H 3650 11366 50  0000 C CNN
+F 1 "7405N" H 3650 11275 50  0000 C CNN
+F 2 "" H 3650 11050 50  0001 C CNN
+F 3 "" H 3650 11050 50  0001 C CNN
+	1    3650 10850
+	1    0    0    -1
+$EndComp
+Wire Wire Line
+	4200 10850 4200 10200
+Wire Wire Line
+	4200 10200 4250 10200
+Wire Wire Line
+	2450 10250 2300 10250
+Wire Wire Line
+	2300 10250 2300 10850
+Wire Wire Line
+	2300 10850 3100 10850
+Wire Wire Line
+	11300 4900 11300 5500
+Text GLabel 11300 4650 0    50   Input ~ 0
+QC1
+$Comp
+L power:+5V #PWR?
+U 1 1 61B91F57
+P 11300 4450
+F 0 "#PWR?" H 11300 4300 50  0001 C CNN
+F 1 "+5V" H 11315 4623 50  0000 C CNN
+F 2 "" H 11300 4450 50  0001 C CNN
+F 3 "" H 11300 4450 50  0001 C CNN
+	1    11300 4450
+	1    0    0    -1
+$EndComp
+Wire Wire Line
+	12400 4550 12550 4550
+Wire Wire Line
+	12550 4550 12550 4850
+Wire Wire Line
+	6900 9500 7150 9500
+$Comp
+L Prinsip:7405N U?
+U 1 1 61BC6AA8
+P 6600 11000
+F 0 "U?" H 6600 11516 50  0000 C CNN
+F 1 "7405N" H 6600 11425 50  0000 C CNN
+F 2 "" H 6600 11200 50  0001 C CNN
+F 3 "" H 6600 11200 50  0001 C CNN
+	1    6600 11000
+	1    0    0    -1
+$EndComp
+Text GLabel 6050 11000 0    50   Input ~ 0
+TO_BUFFER_1
+Wire Wire Line
+	7150 9700 7150 11000
+Text GLabel 7650 9500 2    50   Input ~ 0
+QT
+Wire Wire Line
+	12200 4900 11300 4900
+$Comp
+L Prinsip:7402N U?
+U 1 1 61B91F5D
+P 11850 4550
+F 0 "U?" H 11850 5016 50  0000 C CNN
+F 1 "7402N" H 11850 4925 50  0000 C CNN
+F 2 "" H 11850 4700 50  0001 C CNN
+F 3 "" H 11850 4700 50  0001 C CNN
+	1    11850 4550
+	1    0    0    -1
+$EndComp
+Wire Wire Line
+	12200 5100 12550 5100
 Wire Bus Line
 	3100 900  3100 3350
@@
 Wire Bus Line
 	1100 900  1100 5000
-$Comp
-L power:+5V #PWR?
-U 1 1 61A21106
-P 3400 8250
-F 0 "#PWR?" H 3400 8100 50  0001 C CNN
-F 1 "+5V" H 3415 8423 50  0000 C CNN
-F 2 "" H 3400 8250 50  0001 C CNN
-F 3 "" H 3400 8250 50  0001 C CNN
-	1    3400 8250
-	1    0    0    -1
-$EndComp
+Text GLabel 12550 4950 0    50   Input ~ 0
+QT
 $EndSCHEMATC

Commit message: Updated
Parts:
- added U?: S3, symbol Prinsip:SW
- added U?: R, symbol Prinsip:R
- added U?: SW1, symbol Prinsip:SW1
Connections:
- net +5V: now also U?.~ (~LOAD), U?.~
- net Earth: now also U?.~, U?.~
- net at U?.~: no longer U?.~ (~LOAD)
- net at U?.9 (Qh): now also U?.2 (A), U?.3 (B)
- net at U?.12 (7Q): now also BAR?.3 (A)
- net at U?.4 (5Q): now also BAR?.1 (A)
- net at U?.7 (6Q): now also BAR?.2 (A)
- net at U?.1, U?.~ (~LOAD): now also U?.~
- new net: U?.~, U?.~ (~LOAD)
- new net: U?.~, U?.~
Changed lines of the file:
@@
 	4200 10200 4250 10200
-Wire Wire Line
-	2450 10250 2300 10250
 Wire Wire Line
 	2300 10250 2300 10850
@@
 Wire Wire Line
 	12200 5100 12550 5100
+Text GLabel 12550 4950 0    50   Input ~ 0
+QT
+Wire Wire Line
+	2350 9500 2450 9500
+Wire Wire Line
+	2450 9600 2350 9600
+Connection ~ 2350 9600
+Wire Wire Line
+	2350 9600 2350 9500
+Wire Wire Line
+	2450 9700 2350 9700
+Connection ~ 2350 9700
+Wire Wire Line
+	2350 9700 2350 9600
+Wire Wire Line
+	2450 9800 2350 9800
+Connection ~ 2350 9800
+Wire Wire Line
+	2350 9800 2350 9700
+Wire Wire Line
+	2450 9950 2350 9950
+Connection ~ 2350 9950
+Wire Wire Line
+	2350 9950 2350 9800
+Wire Wire Line
+	2450 10050 2350 10050
+Connection ~ 2350 10050
+Wire Wire Line
+	2350 10050 2350 9950
+Wire Wire Line
+	2450 10150 2350 10150
+Wire Wire Line
+	2350 10150 2350 10050
+Text GLabel 2350 9400 1    50   Input ~ 0
++5V
+Connection ~ 2350 9500
+Wire Wire Line
+	2350 9400 2350 9500
+Wire Wire Line
+	2300 10250 2450 10250
+$Comp
+L Prinsip:SW U?
+U 1 1 61C45C7A
+P 2150 10100
+F 0 "U?" H 2150 10267 50  0001 C CNN
+F 1 "S3" H 2150 10175 50  0000 C CNN
+F 2 "" H 2150 10100 50  0001 C CNN
+F 3 "" H 2150 10100 50  0001 C CNN
+	1    2150 10100
+	1    0    0    -1
+$EndComp
+$Comp
+L power:Earth #PWR?
+U 1 1 61C5AE8B
+P 2000 10250
+F 0 "#PWR?" H 2000 10000 50  0001 C CNN
+F 1 "Earth" H 2000 10100 50  0001 C CNN
+F 2 "" H 2000 10250 50  0001 C CNN
+F 3 "~" H 2000 10250 50  0001 C CNN
+	1    2000 10250
+	1    0    0    -1
+$EndComp
+Wire Wire Line
+	2000 10150 2000 9800
+Wire Wire Line
+	2000 9800 2350 9800
+$Comp
+L power:Earth #PWR?
+U 1 1 61C7552E
+P 2550 11250
+F 0 "#PWR?" H 2550 11000 50  0001 C CNN
+F 1 "Earth" H 2550 11100 50  0001 C CNN
+F 2 "" H 2550 11250 50  0001 C CNN
+F 3 "~" H 2550 11250 50  0001 C CNN
+	1    2550 11250
+	1    0    0    -1
+$EndComp
+$Comp
+L Prinsip:R U?
+U 1 1 61C8D271
+P 2250 11150
+F 0 "U?" H 2250 11275 50  0000 C CNN
+F 1 "R" H 2250 11184 50  0000 C CNN
+F 2 "" H 2250 11150 50  0001 C CNN
+F 3 "" H 2250 11150 50  0001 C CNN
+	1    2250 11150
+	1    0    0    -1
+$EndComp
+$Comp
+L Prinsip:SW1 U?
+U 1 1 61C98DF7
+P 1550 11050
+F 0 "U?" H 1550 11165 50  0000 C CNN
+F 1 "SW1" H 1550 11074 50  0000 C CNN
+F 2 "" H 1550 11050 50  0001 C CNN
+F 3 "" H 1550 11050 50  0001 C CNN
+	1    1550 11050
+	1    0    0    -1
+$EndComp
 Wire Bus Line
 	3100 900  3100 3350
@@
 Wire Bus Line
 	1100 900  1100 5000
-Text GLabel 12550 4950 0    50   Input ~ 0
-QT
 $EndSCHEMATC
