File: Prinsip/Prinsip.sch (KiCad schematic (older format))
At the start: 42 parts

Commit message: upd
Parts:
- removed U?: 74ALS11AM, symbol Prinsip:74ALS11AM
- removed U?: S8, symbol Prinsip:SW
- removed U?: S7, symbol Prinsip:SW
- removed U?: S6, symbol Prinsip:SW
- removed U?: S5, symbol Prinsip:SW
- removed U?: S4, symbol Prinsip:SW
- removed U? (x2): S3, symbol Prinsip:SW
- removed U?: S2, symbol Prinsip:SW
- removed U?: S1, symbol Prinsip:SW
- added R1, R2: R_Small-Device, symbol Принципиально-rescue:R_Small-Device
- added SW2: SW_DPDT_x2, symbol Switch:SW_DPDT_x2
- added U?: TAB-Prinsip, symbol Принципиально-rescue:TAB-Prinsip
- added U?: 7405N, symbol Prinsip:7405N
- added ZQ1: Resonator-Device, symbol Принципиально-rescue:Resonator-Device
- R1: renamed from U?; value R -> 10k
Connections:
- net labels added: A1, CLK, SHIFT_CLR
- net labels removed: TO_BUFFER_1
- wire segments 172 -> 159
Other:
- note removed: "CLK"
- note removed: "GND"
- note removed: "SHIFT_CLR"
- note removed: "VCC"
- moved on the sheet: R1

Commit message: upd
Parts:
- added SW3: SW_DPDT_x2, symbol Switch:SW_DPDT_x2
Connections:
- net +5V: now also SW3.1 (A)
- net Earth: now also SW3.3 (C)
- net at U?.12 (7Q): now also BAR?.3 (A)
- net at U?.4 (5Q): now also BAR?.1 (A)
- net at U?.7 (6Q): now also BAR?.2 (A)
- net at U?.15 (~CLR): now also SW3.2 (B)
- new net: R1.~, U?.~, U?.~ (~LOAD)
Changed lines of the file:
@@
 Wire Wire Line
 	3400 5000 3500 5000
+$Comp
+L Switch:SW_DPDT_x2 SW3
+U 1 1 616811AA
+P 4050 10100
+F 0 "SW3" H 4050 10293 50  0000 C CNN
+F 1 "SW_DPDT_x2" H 4050 10294 50  0001 C CNN
+F 2 "" H 4050 10100 50  0001 C CNN
+F 3 "~" H 4050 10100 50  0001 C CNN
+	1    4050 10100
+	-1   0    0    -1
+$EndComp
 Wire Wire Line
 	4150 2600 4150 3350
+$Comp
+L power:Earth #PWR?
+U 1 1 61689F33
+P 3850 10200
+F 0 "#PWR?" H 3850 9950 50  0001 C CNN
+F 1 "Earth" H 3850 10050 50  0001 C CNN
+F 2 "" H 3850 10200 50  0001 C CNN
+F 3 "~" H 3850 10200 50  0001 C CNN
+	1    3850 10200
+	1    0    0    -1
+$EndComp
+$Comp
+L power:+5V #PWR?
+U 1 1 6168AD22
+P 3850 10000
+F 0 "#PWR?" H 3850 9850 50  0001 C CNN
+F 1 "+5V" H 3865 10173 50  0000 C CNN
+F 2 "" H 3850 10000 50  0001 C CNN
+F 3 "" H 3850 10000 50  0001 C CNN
+	1    3850 10000
+	1    0    0    -1
+$EndComp
 $EndSCHEMATC

Commit message: Added caps
Parts:
- added С1, С2..С11: con-Prinsip, symbol Принципиально-rescue:con-Prinsip
Connections:
- net at U?.12 (7Q): now also BAR?.3 (A)
- net at U?.4 (5Q): now also BAR?.1 (A)
- net at U?.7 (6Q): now also BAR?.2 (A)
- new net: С1.~, С2..С11.~ (x2)
- new net: R1.~, U?.~, U?.~ (~LOAD)
Other:
- note added: "+"
Changed lines of the file:
@@
 	-1   0    0    -1
 $EndComp
-Wire Wire Line
-	4150 2600 4150 3350
 $Comp
 L power:Earth #PWR?
@@
 	1    0    0    -1
 $EndComp
+$Comp
+L Принципиально-rescue:con-Prinsip С1
+U 1 1 61687866
+P 3450 6750
+F 0 "С1" H 3425 6833 50  0000 C CNN
+F 1 "con-Prinsip" H 3425 6834 50  0001 C CNN
+F 2 "" H 3500 7050 50  0001 C CNN
+F 3 "" H 3500 7050 50  0001 C CNN
+	1    3450 6750
+	1    0    0    -1
+$EndComp
+$Comp
+L Принципиально-rescue:con-Prinsip С2..С11
+U 1 1 61688A5C
+P 3450 7100
+F 0 "С2..С11" H 3425 7183 50  0000 C CNN
+F 1 "con-Prinsip" H 3425 7184 50  0001 C CNN
+F 2 "" H 3500 7400 50  0001 C CNN
+F 3 "" H 3500 7400 50  0001 C CNN
+	1    3450 7100
+	1    0    0    -1
+$EndComp
+Wire Wire Line
+	3300 7150 3200 7150
+Wire Wire Line
+	3200 7150 3200 6800
+Wire Wire Line
+	3200 6600 3100 6600
+Wire Wire Line
+	3300 6800 3200 6800
+Connection ~ 3200 6800
+Wire Wire Line
+	3200 6800 3200 6600
+Wire Wire Line
+	3100 6450 3650 6450
+Wire Wire Line
+	3650 6450 3650 6800
+Wire Wire Line
+	3650 7150 3550 7150
+Wire Wire Line
+	3550 6800 3650 6800
+Wire Wire Line
+	4150 2600 4150 3350
+Connection ~ 3650 6800
+Wire Wire Line
+	3650 6800 3650 7150
+Text Notes 3500 6750 0    50   ~ 0
++
 $EndSCHEMATC

Commit message: Fixed DD
Parts:
- removed С1, С2..С11: con-Prinsip, symbol Принципиально-rescue:con-Prinsip
- DD26: renamed from U?; symbol 4xxx_IEEE:4512 -> Prinsip-rescue:4512-4xxx_IEEE
- gave numbers to parts that had none: 27
- renumbered R1 to R3
Connections:
- net at DD6.12 (7Q): now also BAR?.3 (A)
- net at DD6.4 (5Q): now also BAR?.1 (A)
- net at DD6.7 (6Q): now also BAR?.2 (A)
- new net: DD24.~ (~LOAD), R3.~, U?.~
Other:
- note removed: "+"
Changed lines of the file:
@@
 Rev ""
 Comp "МГТУ им. Н.Э. Баумана\\nгруппа ИУ6-64Б"
-Comment1 "Код Баркера"
+Comment1 "Кодировщик кодом Баркера"
 Comment2 "Рожнов В.Д."
 Comment3 "Захаров М.А."
@@
 $EndDescr
 $Comp
-L Prinsip:7410N U?
+L Prinsip:7410N DD9
 U 1 1 6166773C
 P 6200 3600
-F 0 "U?" H 6200 4016 50  0000 C CNN
+F 0 "DD9" H 6200 4016 50  0000 C CNN
 F 1 "7410N" H 6200 3925 50  0000 C CNN
 F 2 "" H 6200 3700 50  0001 C CNN
@@
 $EndComp
 $Comp
-L Prinsip:7408J U?
+L Prinsip:7408J DD7
 U 1 1 6167545D
 P 2500 3650
-F 0 "U?" H 2500 4066 50  0000 C CNN
+F 0 "DD7" H 2500 4066 50  0000 C CNN
 F 1 "7408J" H 2500 3975 50  0000 C CNN
 F 2 "" H 2500 3750 50  0001 C CNN
@@
 $EndComp
 $Comp
-L Prinsip:7405N U?
+L Prinsip:7405N DD19
 U 1 1 61676BE0
 P 7550 6350
-F 0 "U?" H 7550 6866 50  0000 C CNN
+F 0 "DD19" H 7550 6866 50  0000 C CNN
 F 1 "7405N" H 7550 6775 50  0000 C CNN
 F 2 "" H 7550 6550 50  0001 C CNN
@@
 $EndComp
 $Comp
-L Prinsip:7405N U?
+L Prinsip:7405N DD21
 U 1 1 61677469
 P 7550 7200
-F 0 "U?" H 7550 7716 50  0000 C CNN
+F 0 "DD21" H 7550 7716 50  0000 C CNN
 F 1 "7405N" H 7550 7625 50  0000 C CNN
 F 2 "" H 7550 7400 50  0001 C CNN
@@
 $EndComp
 $Comp
-L Prinsip:7410N U?
+L Prinsip:7410N DD20
 U 1 1 616781C6
 P 9400 6100
-F 0 "U?" H 9400 6516 50  0000 C CNN
+F 0 "DD20" H 9400 6516 50  0000 C CNN
 F 1 "7410N" H 9400 6425 50  0000 C CNN
 F 2 "" H 9400 6200 50  0001 C CNN
@@
 $EndComp
 $Comp
-L Prinsip:7405N U?
+L Prinsip:7405N DD12
 U 1 1 61679C6F
 P 9400 4900
-F 0 "U?" H 9400 5416 50  0000 C CNN
+F 0 "DD12" H 9400 5416 50  0000 C CNN
 F 1 "7405N" H 9400 5325 50  0000 C CNN
 F 2 "" H 9400 5100 50  0001 C CNN
@@
 $EndComp
 $Comp
-L Prinsip:7410N U?
+L Prinsip:7410N DD15
 U 1 1 6167AB47
 P 10700 5500
-F 0 "U?" H 10700 5916 50  0000 C CNN
+F 0 "DD15" H 10700 5916 50  0000 C CNN
 F 1 "7410N" H 10700 5825 50  0000 C CNN
 F 2 "" H 10700 5600 50  0001 C CNN
@@
 $EndComp
 $Comp
-L Prinsip:7405N U?
+L Prinsip:7405N DD16
 U 1 1 6167B68A
 P 11850 5500
-F 0 "U?" H 11850 6016 50  0000 C CNN
+F 0 "DD16" H 11850 6016 50  0000 C CNN
 F 1 "7405N" H 11850 5925 50  0000 C CNN
 F 2 "" H 11850 5700 50  0001 C CNN
@@
 $EndComp
 $Comp
-L Prinsip:74F164D U?
+L Prinsip:74F164D DD18
 U 1 1 616815DE
 P 14600 5250
-F 0 "U?" H 14600 5966 50  0000 C CNN
+F 0 "DD18" H 14600 5966 50  0000 C CNN
 F 1 "74F164D" H 14600 5875 50  0000 C CNN
 F 2 "" H 14650 5850 50  0001 C CNN
@@
 $EndComp
 $Comp
-L Prinsip:74F164D U?
+L Prinsip:74F164D DD22
 U 1 1 61683A40
 P 14600 6900
-F 0 "U?" H 14600 7616 50  0000 C CNN
+F 0 "DD22" H 14600 7616 50  0000 C CNN
 F 1 "74F164D" H 14600 7525 50  0000 C CNN
 F 2 "" H 14650 7500 50  0001 C CNN
@@
 	10050 6100 9900 6100
 $Comp
-L Prinsip:7410N U?
+L Prinsip:7410N DD14
 U 1 1 616792E6
 P 8950 5500
-F 0 "U?" H 8950 5916 50  0000 C CNN
+F 0 "DD14" H 8950 5916 50  0000 C CNN
 F 1 "7410N" H 8950 5825 50  0000 C CNN
 F 2 "" H 8950 5600 50  0001 C CNN
@@
 $EndComp
 $Comp
-L Prinsip:7405N U?
+L Prinsip:7405N DD13
 U 1 1 61675F5B
 P 7550 5500
-F 0 "U?" H 7550 6016 50  0000 C CNN
+F 0 "DD13" H 7550 6016 50  0000 C CNN
 F 1 "7405N" H 7550 5925 50  0000 C CNN
 F 2 "" H 7550 5700 50  0001 C CNN
@@
 	5200 3300 5250 3300
 $Comp
-L Prinsip:74ALS21AM U?
+L Prinsip:74ALS21AM DD3
 U 1 1 6166F230
 P 6200 2350
-F 0 "U?" H 6200 2766 50  0000 C CNN
+F 0 "DD3" H 6200 2766 50  0000 C CNN
 F 1 "74ALS21AM" H 6200 2675 50  0000 C CNN
 F 2 "" H 6200 2450 50  0001 C CNN
@@
 QA
 $Comp
-L Prinsip:74273DW U?
+L Prinsip:74273DW DD2
 U 1 1 618BBFDD
 P 11800 1600
-F 0 "U?" H 11800 2316 50  0000 C CNN
+F 0 "DD2" H 11800 2316 50  0000 C CNN
 F 1 "74273DW" H 11800 2225 50  0000 C CNN
 F 2 "" H 11850 2200 50  0001 C CNN
@@
 $EndComp
 $Comp
-L Prinsip:74273DW U?
+L Prinsip:74273DW DD6
 U 1 1 618BD466
 P 11800 3200
-F 0 "U?" H 11800 3916 50  0000 C CNN
+F 0 "DD6" H 11800 3916 50  0000 C CNN
 F 1 "74273DW" H 11800 3825 50  0000 C CNN
 F 2 "" H 11850 3800 50  0001 C CNN
@@
 	10850 3800 11250 3800
 $Comp
-L Prinsip:7405N U?
+L Prinsip:7405N DD4
 U 1 1 618EAB2F
 P 10300 3000
-F 0 "U?" H 10300 3516 50  0000 C CNN
+F 0 "DD4" H 10300 3516 50  0000 C CNN
 F 1 "7405N" H 10300 3425 50  0000 C CNN
 F 2 "" H 10300 3200 50  0001 C CNN
@@
 $EndComp
 $Comp
-L Prinsip:74163N U?
+L Prinsip:74163N DD24
 U 1 1 6196D97B
 P 2800 9300
-F 0 "U?" H 2850 9365 50  0000 C CNN
+F 0 "DD24" H 2850 9365 50  0000 C CNN
 F 1 "74163N" H 2850 9274 50  0000 C CNN
 F 2 "" H 2800 9300 50  0001 C CNN
@@
 $EndComp
 $Comp
-L Prinsip:74F164D U?
+L Prinsip:74F164D DD25
 U 1 1 6196E84B
 P 4800 9650
-F 0 "U?" H 4800 10366 50  0000 C CNN
+F 0 "DD25" H 4800 10366 50  0000 C CNN
 F 1 "74F164D" H 4800 10275 50  0000 C CNN
 F 2 "" H 4850 10250 50  0001 C CNN
@@
 $EndComp
 $Comp
-L 4xxx_IEEE:4512 U?
+L Prinsip-rescue:4512-4xxx_IEEE DD26
 U 1 1 6196F3A5
 P 6350 9500
-F 0 "U?" H 6350 10366 50  0000 C CNN
+F 0 "DD26" H 6350 10366 50  0000 C CNN
 F 1 "4512BD" H 6350 10275 50  0000 C CNN
 F 2 "" H 6350 9500 50  0001 C CNN
@@
 Connection ~ 4250 9500
 $Comp
-L Prinsip:7474N U?
+L Prinsip:7474N DD27
 U 1 1 619D0C4B
 P 7400 9600
-F 0 "U?" H 7400 10031 50  0000 C CNN
+F 0 "DD27" H 7400 10031 50  0000 C CNN
 F 1 "7474N" H 7400 9940 50  0000 C CNN
 F 2 "" H 7400 9600 50  0001 C CNN
@@
 	1    0    0    -1
 $EndComp
-Text GLabel 3250 9700 2    50   Input ~ 0
+Text GLabel 3250 9600 2    50   Input ~ 0
 QC1
 $Comp
-L Prinsip:74163N U?
+L Prinsip:74163N DD23
 U 1 1 61A3EC68
 P 4800 7700
-F 0 "U?" H 4850 7765 50  0000 C CNN
+F 0 "DD23" H 4850 7765 50  0000 C CNN
 F 1 "74163N" H 4850 7674 50  0000 C CNN
 F 2 "" H 4800 7700 50  0001 C CNN
@@
 	5750 8900 5750 8700
 $Comp
-L Prinsip:7405N U?
+L Prinsip:7405N DD28
 U 1 1 61B006B1
 P 3650 10850
-F 0 "U?" H 3650 11366 50  0000 C CNN
+F 0 "DD28" H 3650 11366 50  0000 C CNN
 F 1 "7405N" H 3650 11275 50  0000 C CNN
 F 2 "" H 3650 11050 50  0001 C CNN
@@
 	6900 9500 7150 9500
 $Comp
-L Prinsip:7405N U?
+L Prinsip:7405N DD29
 U 1 1 61BC6AA8
 P 6600 11000
-F 0 "U?" H 6600 11516 50  0000 C CNN
+F 0 "DD29" H 6600 11516 50  0000 C CNN
 F 1 "7405N" H 6600 11425 50  0000 C CNN
 F 2 "" H 6600 11200 50  0001 C CNN
@@
 	12200 4900 11300 4900
 $Comp
-L Prinsip:7402N U?
+L Prinsip:7402N DD1
 U 1 1 61B91F5D
 P 11850 4550
-F 0 "U?" H 11850 5016 50  0000 C CNN
+F 0 "DD1" H 11850 5016 50  0000 C CNN
 F 1 "7402N" H 11850 4925 50  0000 C CNN
 F 2 "" H 11850 4700 50  0001 C CNN
@@
 $EndComp
 $Comp
-L Prinsip:R R1
+L Prinsip:R R3
 U 1 1 61C8D271
 P 2800 11150
-F 0 "R1" H 2800 11275 50  0000 C CNN
+F 0 "R3" H 2800 11275 50  0000 C CNN
 F 1 "10k" H 2800 11184 50  0000 C CNN
 F 2 "" H 2800 11150 50  0001 C CNN
@@
 L Принципиально-rescue:TAB-Prinsip U?
 U 1 1 6167FD6B
-P 2200 6800
-F 0 "U?" H 3128 7170 50  0001 L CNN
-F 1 "TAB-Prinsip" H 3128 7124 50  0001 L CNN
-F 2 "" H 850 7900 50  0001 C CNN
-F 3 "" H 850 7900 50  0001 C CNN
-	1    2200 6800
+P 2250 6900
+F 0 "U?" H 3178 7270 50  0001 L CNN
+F 1 "TAB-Prinsip" H 3178 7224 50  0001 L CNN
+F 2 "" H 900 8000 50  0001 C CNN
+F 3 "" H 900 8000 50  0001 C CNN
+	1    2250 6900
 	1    0    0    -1
 $EndComp
@@
 +5V
 $Comp
-L Prinsip:7432N U?
+L Prinsip:7432N DD8
 U 1 1 61674B22
 P 3750 3550
-F 0 "U?" H 3750 3966 50  0000 C CNN
+F 0 "DD8" H 3750 3966 50  0000 C CNN
 F 1 "7432N" H 3750 3875 50  0000 C CNN
 F 2 "" H 3750 3650 50  0001 C CNN
@@
 $EndComp
 $Comp
-L Prinsip:74163N U?
+L Prinsip:74163N DD5
 U 1 1 6166D0AD
 P 4750 2700
-F 0 "U?" H 4692 2765 50  0000 C CNN
+F 0 "DD5" H 4692 2765 50  0000 C CNN
 F 1 "74163N" H 4692 2674 50  0000 C CNN
 F 2 "" H 4750 2700 50  0001 C CNN
@@
 A1
 $Comp
-L Prinsip:7405N U?
+L Prinsip:7405N DD1
 U 1 1 61689988
 P 7600 1300
-F 0 "U?" H 7600 1816 50  0000 C CNN
+F 0 "DD1" H 7600 1816 50  0000 C CNN
 F 1 "7405N" H 7600 1725 50  0000 C CNN
 F 2 "" H 7600 1500 50  0001 C CNN
@@
 +5V
 $Comp
-L Prinsip:74157N U?
+L Prinsip:74157N DD17
 U 1 1 6167DF8D
 P 13100 5250
-F 0 "U?" H 13100 5966 50  0000 C CNN
+F 0 "DD17" H 13100 5966 50  0000 C CNN
 F 1 "74157N" H 13100 5875 50  0000 C CNN
 F 2 "" H 13150 5850 50  0001 C CNN
@@
 $EndComp
 $Comp
-L Prinsip:7405N U?
+L Prinsip:7405N DD10
 U 1 1 6187BF3E
 P 2850 5000
-F 0 "U?" H 2850 5516 50  0000 C CNN
+F 0 "DD10" H 2850 5516 50  0000 C CNN
 F 1 "7405N" H 2850 5425 50  0000 C CNN
 F 2 "" H 2850 5200 50  0001 C CNN
@@
 	1    0    0    -1
 $EndComp
-$Comp
-L Принципиально-rescue:con-Prinsip С1
-U 1 1 61687866
-P 3450 6750
-F 0 "С1" H 3425 6833 50  0000 C CNN
-F 1 "con-Prinsip" H 3425 6834 50  0001 C CNN
-F 2 "" H 3500 7050 50  0001 C CNN
-F 3 "" H 3500 7050 50  0001 C CNN
-	1    3450 6750
-	1    0    0    -1
-$EndComp
-$Comp
-L Принципиально-rescue:con-Prinsip С2..С11
-U 1 1 61688A5C
-P 3450 7100
-F 0 "С2..С11" H 3425 7183 50  0000 C CNN
-F 1 "con-Prinsip" H 3425 7184 50  0001 C CNN
-F 2 "" H 3500 7400 50  0001 C CNN
-F 3 "" H 3500 7400 50  0001 C CNN
-	1    3450 7100
-	1    0    0    -1
-$EndComp
-Wire Wire Line
-	3300 7150 3200 7150
-Wire Wire Line
-	3200 7150 3200 6800
-Wire Wire Line
-	3200 6600 3100 6600
-Wire Wire Line
-	3300 6800 3200 6800
-Connection ~ 3200 6800
-Wire Wire Line
-	3200 6800 3200 6600
-Wire Wire Line
-	3100 6450 3650 6450
-Wire Wire Line
-	3650 6450 3650 6800
-Wire Wire Line
-	3650 7150 3550 7150
-Wire Wire Line
-	3550 6800 3650 6800
 Wire Wire Line
 	4150 2600 4150 3350
-Connection ~ 3650 6800
-Wire Wire Line
-	3650 6800 3650 7150
-Text Notes 3500 6750 0    50   ~ 0
-+
 $EndSCHEMATC

Commit message: Added caps + DD
Parts:
- added C1, C2..C11: con-Prinsip, symbol Принципиально-rescue:con-Prinsip
Connections:
- net at DD6.12 (7Q): now also BAR?.3 (A)
- net at DD6.4 (5Q): now also BAR?.1 (A)
- net at DD6.7 (6Q): now also BAR?.2 (A)
- new net: C1.~, C2..C11.~ (x2)
- new net: DD24.~ (~LOAD), R3.~, U?.~
Other:
- note added: "+"
Changed lines of the file:
@@
+	1    0    0    -1
+$EndComp
+$Comp
+L Принципиально-rescue:con-Prinsip C1
+U 1 1 616875C2
+P 3550 6850
+F 0 "C1" H 3525 6933 50  0000 C CNN
+F 1 "con-Prinsip" H 3525 6934 50  0001 C CNN
+F 2 "" H 3600 7150 50  0001 C CNN
+F 3 "" H 3600 7150 50  0001 C CNN
+	1    3550 6850
+	1    0    0    -1
+$EndComp
+$Comp
+L Принципиально-rescue:con-Prinsip C2..C11
+U 1 1 61687D14
+P 3550 7250
+F 0 "C2..C11" H 3525 7333 50  0000 C CNN
+F 1 "con-Prinsip" H 3525 7334 50  0001 C CNN
+F 2 "" H 3600 7550 50  0001 C CNN
+F 3 "" H 3600 7550 50  0001 C CNN
+	1    3550 7250
 	1    0    0    -1
 $EndComp
 Wire Wire Line
+	3150 6750 3250 6750
+Wire Wire Line
+	3250 6750 3250 6900
+Wire Wire Line
+	3250 7300 3400 7300
+Wire Wire Line
+	3400 6900 3250 6900
+Connection ~ 3250 6900
+Wire Wire Line
+	3250 6900 3250 7300
+Wire Wire Line
+	3150 6550 3850 6550
+Wire Wire Line
+	3850 6550 3850 6900
+Wire Wire Line
+	3850 7300 3650 7300
+Wire Wire Line
+	3650 6900 3850 6900
+Wire Wire Line
 	4150 2600 4150 3350
+Connection ~ 3850 6900
+Wire Wire Line
+	3850 6900 3850 7300
+Text Notes 3700 6850 0    50   ~ 0
++
 $EndSCHEMATC

Commit message: Updated pdf
Parts:
- renumbered C2..C11 to C2..C12
Connections:
- net at DD6.12 (7Q): now also BAR?.3 (A)
- net at DD6.4 (5Q): now also BAR?.1 (A)
- net at DD6.7 (6Q): now also BAR?.2 (A)
- new net: C1.~, C2..C12.~
- new net: DD24.~ (~LOAD), R3.~, U?.~
Other:
- note added: "Контакт 16 микросхем\nDD2, DD5, DD6, DD17, DD18,\nDD22, DD23, DD24, DD25, DD26, DD27\nподключить к VCC"
- note added: "Контакт 8 микросхем\nDD2, DD5, DD6, DD17, DD18,\nDD22, DD23, DD24, DD25, DD26, DD27\nПодключить к GND"
Changed lines of the file:
@@
 $EndComp
 $Comp
-L Принципиально-rescue:con-Prinsip C2..C11
+L Принципиально-rescue:con-Prinsip C2..C12
 U 1 1 61687D14
 P 3550 7250
-F 0 "C2..C11" H 3525 7333 50  0000 C CNN
+F 0 "C2..C12" H 3525 7333 50  0000 C CNN
 F 1 "con-Prinsip" H 3525 7334 50  0001 C CNN
 F 2 "" H 3600 7550 50  0001 C CNN
@@
 Wire Wire Line
 	3650 6900 3850 6900
-Wire Wire Line
-	4150 2600 4150 3350
 Connection ~ 3850 6900
 Wire Wire Line
@@
 Text Notes 3700 6850 0    50   ~ 0
 +
+Text Notes 1750 7600 0    50   ~ 0
+Контакт 16 микросхем\nDD2, DD5, DD6, DD17, DD18,\nDD22, DD23, DD24, DD25, DD26, DD27\nподключить к VCC
+Text Notes 1750 8100 0    50   ~ 0
+Контакт 8 микросхем\nDD2, DD5, DD6, DD17, DD18,\nDD22, DD23, DD24, DD25, DD26, DD27\nПодключить к GND
+Wire Wire Line
+	4150 2600 4150 3350
 $EndSCHEMATC
