File: Prinsip/Prinsip.sch (KiCad schematic (older format))
At the start: 41 parts, among them SW2 SW_DPDT_x2, SW3 SW_DPDT_x2

Commit message: Updated pdf
Parts:
- renumbered DD7 to DD1, DD9 to DD10, DD26 to DD11, DD29 to DD12, DD1 to DD13, DD13 to DD14, DD19 to DD15, DD21 to DD16, DD27 to DD17, DD14 to DD18, DD12 to DD19, DD10 to DD2, DD4 to DD21, DD15 to DD22, DD2 to DD23, DD6 to DD24, DD1 to DD25, DD16 to DD26, DD17 to DD27, DD18 to DD28, DD22 to DD29, DD24 to DD3, DD8 to DD4, DD28 to DD5, DD5 to DD6, DD23 to DD7, DD25 to DD8, DD3 to DD9
Connections:
- net at DD24.12 (7Q): now also BAR?.3 (A)
- net at DD24.4 (5Q): now also BAR?.1 (A)
- net at DD24.7 (6Q): now also BAR?.2 (A)
- new net: C1.~, C2..C12.~
- new net: DD3.~ (~LOAD), R3.~, U?.~
Other:
- note added: "Контакт 16 микросхем\nDD3, DDDD6, DD7, DD8, DD11, DD17,\nDD23, DD24, DD27, DD28, DD29\nподключить к VCC"
- note added: "Контакт 8 микросхем\nDD3, DDDD6, DD7, DD8, DD11, DD17,\nDD23, DD24, DD27, DD28, DD29\nПодключить к GND"
- note removed: "Контакт 16 микросхем\nDD2, DD5, DD6, DD17, DD18,\nDD22, DD23, DD24, DD25, DD26, DD27\nподключить к VCC"
- note removed: "Контакт 8 микросхем\nDD2, DD5, DD6, DD17, DD18,\nDD22, DD23, DD24, DD25, DD26, DD27\nПодключить к GND"
Changed lines of the file:
@@
 $EndDescr
 $Comp
-L Prinsip:7410N DD9
+L Prinsip:7410N DD10
 U 1 1 6166773C
 P 6200 3600
-F 0 "DD9" H 6200 4016 50  0000 C CNN
+F 0 "DD10" H 6200 4016 50  0000 C CNN
 F 1 "7410N" H 6200 3925 50  0000 C CNN
 F 2 "" H 6200 3700 50  0001 C CNN
@@
 $EndComp
 $Comp
-L Prinsip:7408J DD7
+L Prinsip:7408J DD1
 U 1 1 6167545D
 P 2500 3650
-F 0 "DD7" H 2500 4066 50  0000 C CNN
+F 0 "DD1" H 2500 4066 50  0000 C CNN
 F 1 "7408J" H 2500 3975 50  0000 C CNN
 F 2 "" H 2500 3750 50  0001 C CNN
@@
 $EndComp
 $Comp
-L Prinsip:7405N DD19
+L Prinsip:7405N DD15
 U 1 1 61676BE0
 P 7550 6350
-F 0 "DD19" H 7550 6866 50  0000 C CNN
+F 0 "DD15" H 7550 6866 50  0000 C CNN
 F 1 "7405N" H 7550 6775 50  0000 C CNN
 F 2 "" H 7550 6550 50  0001 C CNN
@@
 $EndComp
 $Comp
-L Prinsip:7405N DD21
+L Prinsip:7405N DD16
 U 1 1 61677469
 P 7550 7200
-F 0 "DD21" H 7550 7716 50  0000 C CNN
+F 0 "DD16" H 7550 7716 50  0000 C CNN
 F 1 "7405N" H 7550 7625 50  0000 C CNN
 F 2 "" H 7550 7400 50  0001 C CNN
@@
 $EndComp
 $Comp
-L Prinsip:7405N DD12
+L Prinsip:7405N DD19
 U 1 1 61679C6F
 P 9400 4900
-F 0 "DD12" H 9400 5416 50  0000 C CNN
+F 0 "DD19" H 9400 5416 50  0000 C CNN
 F 1 "7405N" H 9400 5325 50  0000 C CNN
 F 2 "" H 9400 5100 50  0001 C CNN
@@
 $EndComp
 $Comp
-L Prinsip:7410N DD15
+L Prinsip:7410N DD22
 U 1 1 6167AB47
 P 10700 5500
-F 0 "DD15" H 10700 5916 50  0000 C CNN
+F 0 "DD22" H 10700 5916 50  0000 C CNN
 F 1 "7410N" H 10700 5825 50  0000 C CNN
 F 2 "" H 10700 5600 50  0001 C CNN
@@
 $EndComp
 $Comp
-L Prinsip:7405N DD16
+L Prinsip:7405N DD26
 U 1 1 6167B68A
 P 11850 5500
-F 0 "DD16" H 11850 6016 50  0000 C CNN
+F 0 "DD26" H 11850 6016 50  0000 C CNN
 F 1 "7405N" H 11850 5925 50  0000 C CNN
 F 2 "" H 11850 5700 50  0001 C CNN
@@
 $EndComp
 $Comp
-L Prinsip:74F164D DD18
+L Prinsip:74F164D DD28
 U 1 1 616815DE
 P 14600 5250
-F 0 "DD18" H 14600 5966 50  0000 C CNN
+F 0 "DD28" H 14600 5966 50  0000 C CNN
 F 1 "74F164D" H 14600 5875 50  0000 C CNN
 F 2 "" H 14650 5850 50  0001 C CNN
@@
 $EndComp
 $Comp
-L Prinsip:74F164D DD22
+L Prinsip:74F164D DD29
 U 1 1 61683A40
 P 14600 6900
-F 0 "DD22" H 14600 7616 50  0000 C CNN
+F 0 "DD29" H 14600 7616 50  0000 C CNN
 F 1 "74F164D" H 14600 7525 50  0000 C CNN
 F 2 "" H 14650 7500 50  0001 C CNN
@@
 	10050 6100 9900 6100
 $Comp
-L Prinsip:7410N DD14
+L Prinsip:7410N DD18
 U 1 1 616792E6
 P 8950 5500
-F 0 "DD14" H 8950 5916 50  0000 C CNN
+F 0 "DD18" H 8950 5916 50  0000 C CNN
 F 1 "7410N" H 8950 5825 50  0000 C CNN
 F 2 "" H 8950 5600 50  0001 C CNN
@@
 $EndComp
 $Comp
-L Prinsip:7405N DD13
+L Prinsip:7405N DD14
 U 1 1 61675F5B
 P 7550 5500
-F 0 "DD13" H 7550 6016 50  0000 C CNN
+F 0 "DD14" H 7550 6016 50  0000 C CNN
 F 1 "7405N" H 7550 5925 50  0000 C CNN
 F 2 "" H 7550 5700 50  0001 C CNN
@@
 	5200 3300 5250 3300
 $Comp
-L Prinsip:74ALS21AM DD3
+L Prinsip:74ALS21AM DD9
 U 1 1 6166F230
 P 6200 2350
-F 0 "DD3" H 6200 2766 50  0000 C CNN
+F 0 "DD9" H 6200 2766 50  0000 C CNN
 F 1 "74ALS21AM" H 6200 2675 50  0000 C CNN
 F 2 "" H 6200 2450 50  0001 C CNN
@@
 QA
 $Comp
-L Prinsip:74273DW DD2
+L Prinsip:74273DW DD23
 U 1 1 618BBFDD
 P 11800 1600
-F 0 "DD2" H 11800 2316 50  0000 C CNN
+F 0 "DD23" H 11800 2316 50  0000 C CNN
 F 1 "74273DW" H 11800 2225 50  0000 C CNN
 F 2 "" H 11850 2200 50  0001 C CNN
@@
 $EndComp
 $Comp
-L Prinsip:74273DW DD6
+L Prinsip:74273DW DD24
 U 1 1 618BD466
 P 11800 3200
-F 0 "DD6" H 11800 3916 50  0000 C CNN
+F 0 "DD24" H 11800 3916 50  0000 C CNN
 F 1 "74273DW" H 11800 3825 50  0000 C CNN
 F 2 "" H 11850 3800 50  0001 C CNN
@@
 	10850 3800 11250 3800
 $Comp
-L Prinsip:7405N DD4
+L Prinsip:7405N DD21
 U 1 1 618EAB2F
 P 10300 3000
-F 0 "DD4" H 10300 3516 50  0000 C CNN
+F 0 "DD21" H 10300 3516 50  0000 C CNN
 F 1 "7405N" H 10300 3425 50  0000 C CNN
 F 2 "" H 10300 3200 50  0001 C CNN
@@
 $EndComp
 $Comp
-L Prinsip:74163N DD24
+L Prinsip:74163N DD3
 U 1 1 6196D97B
 P 2800 9300
-F 0 "DD24" H 2850 9365 50  0000 C CNN
+F 0 "DD3" H 2850 9365 50  0000 C CNN
 F 1 "74163N" H 2850 9274 50  0000 C CNN
 F 2 "" H 2800 9300 50  0001 C CNN
@@
 $EndComp
 $Comp
-L Prinsip:74F164D DD25
+L Prinsip:74F164D DD8
 U 1 1 6196E84B
 P 4800 9650
-F 0 "DD25" H 4800 10366 50  0000 C CNN
+F 0 "DD8" H 4800 10366 50  0000 C CNN
 F 1 "74F164D" H 4800 10275 50  0000 C CNN
 F 2 "" H 4850 10250 50  0001 C CNN
@@
 $EndComp
 $Comp
-L Prinsip-rescue:4512-4xxx_IEEE DD26
+L Prinsip-rescue:4512-4xxx_IEEE DD11
 U 1 1 6196F3A5
 P 6350 9500
-F 0 "DD26" H 6350 10366 50  0000 C CNN
+F 0 "DD11" H 6350 10366 50  0000 C CNN
 F 1 "4512BD" H 6350 10275 50  0000 C CNN
 F 2 "" H 6350 9500 50  0001 C CNN
@@
 Connection ~ 4250 9500
 $Comp
-L Prinsip:7474N DD27
+L Prinsip:7474N DD17
 U 1 1 619D0C4B
 P 7400 9600
-F 0 "DD27" H 7400 10031 50  0000 C CNN
+F 0 "DD17" H 7400 10031 50  0000 C CNN
 F 1 "7474N" H 7400 9940 50  0000 C CNN
 F 2 "" H 7400 9600 50  0001 C CNN
@@
 QC1
 $Comp
-L Prinsip:74163N DD23
+L Prinsip:74163N DD7
 U 1 1 61A3EC68
 P 4800 7700
-F 0 "DD23" H 4850 7765 50  0000 C CNN
+F 0 "DD7" H 4850 7765 50  0000 C CNN
 F 1 "74163N" H 4850 7674 50  0000 C CNN
 F 2 "" H 4800 7700 50  0001 C CNN
@@
 	5750 8900 5750 8700
 $Comp
-L Prinsip:7405N DD28
+L Prinsip:7405N DD5
 U 1 1 61B006B1
 P 3650 10850
-F 0 "DD28" H 3650 11366 50  0000 C CNN
+F 0 "DD5" H 3650 11366 50  0000 C CNN
 F 1 "7405N" H 3650 11275 50  0000 C CNN
 F 2 "" H 3650 11050 50  0001 C CNN
@@
 	6900 9500 7150 9500
 $Comp
-L Prinsip:7405N DD29
+L Prinsip:7405N DD12
 U 1 1 61BC6AA8
 P 6600 11000
-F 0 "DD29" H 6600 11516 50  0000 C CNN
+F 0 "DD12" H 6600 11516 50  0000 C CNN
 F 1 "7405N" H 6600 11425 50  0000 C CNN
 F 2 "" H 6600 11200 50  0001 C CNN
@@
 	12200 4900 11300 4900
 $Comp
-L Prinsip:7402N DD1
+L Prinsip:7402N DD25
 U 1 1 61B91F5D
 P 11850 4550
-F 0 "DD1" H 11850 5016 50  0000 C CNN
+F 0 "DD25" H 11850 5016 50  0000 C CNN
 F 1 "7402N" H 11850 4925 50  0000 C CNN
 F 2 "" H 11850 4700 50  0001 C CNN
@@
 +5V
 $Comp
-L Prinsip:7432N DD8
+L Prinsip:7432N DD4
 U 1 1 61674B22
 P 3750 3550
-F 0 "DD8" H 3750 3966 50  0000 C CNN
+F 0 "DD4" H 3750 3966 50  0000 C CNN
 F 1 "7432N" H 3750 3875 50  0000 C CNN
 F 2 "" H 3750 3650 50  0001 C CNN
@@
 $EndComp
 $Comp
-L Prinsip:74163N DD5
+L Prinsip:74163N DD6
 U 1 1 6166D0AD
 P 4750 2700
-F 0 "DD5" H 4692 2765 50  0000 C CNN
+F 0 "DD6" H 4692 2765 50  0000 C CNN
 F 1 "74163N" H 4692 2674 50  0000 C CNN
 F 2 "" H 4750 2700 50  0001 C CNN
@@
 A1
 $Comp
-L Prinsip:7405N DD1
+L Prinsip:7405N DD13
 U 1 1 61689988
 P 7600 1300
-F 0 "DD1" H 7600 1816 50  0000 C CNN
+F 0 "DD13" H 7600 1816 50  0000 C CNN
 F 1 "7405N" H 7600 1725 50  0000 C CNN
 F 2 "" H 7600 1500 50  0001 C CNN
@@
 +5V
 $Comp
-L Prinsip:74157N DD17
+L Prinsip:74157N DD27
 U 1 1 6167DF8D
 P 13100 5250
-F 0 "DD17" H 13100 5966 50  0000 C CNN
+F 0 "DD27" H 13100 5966 50  0000 C CNN
 F 1 "74157N" H 13100 5875 50  0000 C CNN
 F 2 "" H 13150 5850 50  0001 C CNN
@@
 $EndComp
 $Comp
-L Prinsip:7405N DD10
+L Prinsip:7405N DD2
 U 1 1 6187BF3E
 P 2850 5000
-F 0 "DD10" H 2850 5516 50  0000 C CNN
+F 0 "DD2" H 2850 5516 50  0000 C CNN
 F 1 "7405N" H 2850 5425 50  0000 C CNN
 F 2 "" H 2850 5200 50  0001 C CNN
@@
 +
 Text Notes 1750 7600 0    50   ~ 0
-Контакт 16 микросхем\nDD2, DD5, DD6, DD17, DD18,\nDD22, DD23, DD24, DD25, DD26, DD27\nподключить к VCC
+Контакт 16 микросхем\nDD3, DDDD6, DD7, DD8, DD11, DD17,\nDD23, DD24, DD27, DD28, DD29\nподключить к VCC
 Text Notes 1750 8100 0    50   ~ 0
-Контакт 8 микросхем\nDD2, DD5, DD6, DD17, DD18,\nDD22, DD23, DD24, DD25, DD26, DD27\nПодключить к GND
+Контакт 8 микросхем\nDD3, DDDD6, DD7, DD8, DD11, DD17,\nDD23, DD24, DD27, DD28, DD29\nПодключить к GND
 Wire Wire Line
 	4150 2600 4150 3350
