File: VD/vd.sch (KiCad schematic (older format))
At the start: 0 parts

Commit message: Added VD
Other:
- note added: "BARKER"
- note added: "REVERSE"
- note added: "Генератор кода Баркера"
- note added: "Последовательность Баркера при REVERSE = 0"
- note added: "Последовательность Баркера при REVERSE = 1"
